File: hardware/eagle/nrfice.sch (EAGLE design)
At the start: 121 parts, among them J1 JLINKNEEDLE6, J10 C27438, J11 C40877, J14 PZ254V-11-04P, J15 PZ254V-11-04P, J16 C30734, J17 PZ254V-11-04P, J2 USB-TYPE-C-020, J3 PZ254V-11-04P, J4 C57369, J5 C35445, J7 DC-050-2.0-B, J8 USB-TYPE-C-020, J9 C30734, T1 MTA1, T10 MTA1, T11 T, T12 T, T13 MTA1, T2 MTA1, T3 MTA1, T4 MTA1, T5 MTA1, T6 T, T7 T, T8 T, T9 T, U1 UHD1110-FKA, U10 AT25SF128A-SHB-T, U2 BT40F, U3 ME6211A33M3G-N, U4 LM1085S-5.0, U5 UHD1110-FKA, U6 ME6206A25XG, U7 ICE40UP5K-SG48I, U8 STM32F072CBU6TR, U9 HX6306P122MR

Commit message: Updates to the android app, cleaned up hardware files, and update to firmware.
Parts:
- removed S1, S6, S7, S8: TS-1091C-A8B3-D2, robotonea1u:TS-1091C-A8B3-D2
- added J6: MTA21, nrfice04:MTA21
- added R40, R41: DNL, nrfice04:R-US_R0402
- added R42: 5.1K, nrfice04:R-US_R0402
- added SW1, SW6, SW7, SW8: TS-1091C-A8B3-D2, nrfice04:TS-1091C-A8B3-D2
- added T14, T15, T16, T17, T18, T19, T20, T21, T22, T23, T24, T27: TT2, nrfice04:TT2
- C1, C10, C11, C14, C15, C16, C17, C18, C19, C2, C20, C21, C23, C31, C32, C34, C48, C5, C6, C62, C63, C65, C67, C68, C69, C7, C70, C71, C75, C8: device robotonea1u:C-USC0402 -> nrfice04:C-USC0402
- C12: value 10uF -> 22uF; device robotonea1u:C-USC0805 -> nrfice04:C-USC0805; DESC 10uF,16V,10%,X5R,0805 -> 22uF,25V,20%,X5R,0805; MPN CL21A106KOQNNNE -> CL21A226MAYNNNE
- C13, C22, C3, C4, C9: device robotonea1u:C-USC0805 -> nrfice04:C-USC0805
- D2: device robotonea1u:PRTR5V0U2X -> nrfice04:PRTR5V0U2X
- D5: device robotonea1u:XL-1608SYGC-06 -> nrfice04:XL-1608SYGC-06
- J1: device robotonea1u:JLINKNEEDLE6 -> nrfice04:JLINKNEEDLE6
- J10: device robotonea1u:C27438 -> nrfice04:C27438
- J11: device robotonea1u:C40877 -> nrfice04:C40877
- J14, J15, J17, J3: device robotonea1u:PZ254V-11-04P -> nrfice04:PZ254V-11-04P
- J16, J9: device robotonea1u:C30734 -> nrfice04:C30734
- J2, J8: device robotonea1u:USB-TYPE-C-020 -> nrfice04:USB-TYPE-C-020
- J4: device robotonea1u:C57369 -> nrfice04:C57369
- J5: device robotonea1u:C35445 -> nrfice04:C35445
- J7: device robotonea1u:DC-050-2.0-B -> nrfice04:DC-050-2.0-B
- L1: device robotonea1u:L-USL0402 -> nrfice04:L-USL0402
- OSC1: device robotonea1u:X1G004171004000 -> nrfice04:X1G004171004000
- R1, R10, R11, R13, R14, R15, R17, R18, R2, R22, R24, R28, R29, R3, R30, R31, R37, R38, R39, R6, R8, R9, R91: device robotonea1u:R-US_R0402 -> nrfice04:R-US_R0402
- R12, R16, R33, R34, R35, R36: device robotonea1u:R-US_R0603 -> nrfice04:R-US_R0603
- R19, R20, R21, R25: device robotonea1u:R-US_R0402 -> nrfice04:R-US_R0402; DESC 5.1K,1%,1/16W,0402 -> 5.1K Ohm,1%,1/16W,0402
- R23, R4: device robotonea1u:R-US_R0402 -> nrfice04:R-US_R0402; MPN RC0402FR-070RL -> RC0402FR-0710KL
- R26, R27, R32: value 10K -> DNL; device robotonea1u:R-US_R0402 -> nrfice04:R-US_R0402; DESC 10K Ohm,1%,1/16W,0402 -> DNL
- R5: value 1K -> 680; device robotonea1u:R-US_R0402 -> nrfice04:R-US_R0402; DESC 1K Ohm,1%,1/16W,0402 -> 680 Ohms,1%,1/16W,0402; MPN RC0402FR-071KL -> RC0402FR-07680RL
- R7: value 680 -> 1K; device robotonea1u:R-US_R0402 -> nrfice04:R-US_R0402; DESC 680 Ohms,1%,1/16W,0402 -> 1K Ohm,1%,1/16W,0402; MPN RC0402FR-07680RL -> RC0402FR-071KL
- T1, T10, T13, T2, T3, T4, T5: device robotonea1u:MTA1 -> nrfice04:MTA1
- T11, T12, T6, T7, T8, T9: device robotonea1u:T -> nrfice04:T
- U1, U5: device robotonea1u:UHD1110-FKA -> nrfice04:UHD1110-FKA
- U10: device robotonea1u:AT25SF128A-SHB-T -> nrfice04:AT25SF128A-SHB-T
- U2: device robotonea1u:BT40F -> nrfice04:BT40F
- U3: device robotonea1u:ME6211A33M3G-N -> nrfice04:ME6211A33M3G-N
- U4: device robotonea1u:LM1085S-5.0 -> nrfice04:LM1085S-5.0
- U6: device robotonea1u:ME6206A25XG -> nrfice04:ME6206A25XG
- U7: device robotonea1u:ICE40UP5K-SG48I -> nrfice04:ICE40UP5K-SG48I
- U8: device robotonea1u:STM32F072CBU6TR -> nrfice04:STM32F072CBU6TR
- U9: device robotonea1u:HX6306P122MR -> nrfice04:HX6306P122MR
Connections:
- removed net NRFICE3: J16.6, U2.4P001, U7.19
- new net AREF: J5.8, R42.1
- new net ICE_19: J16.6, U7.19
- new net P0XL1: R40.1, U2.3P000
- new net P1XL2: R40.2, U2.4P001
- net 3V3: now also R42.2, T15.T; no longer J5.8
- net 9V: now also J6.2
- net ARD_D2: now also J9.12, U7.20GBIN3; no longer J9.6, U2.C3P024, U7.43
- net ARD_D3: now also J9.10, U2.C1P031, U7.38; no longer J9.8, U2.C2P021, U7.42
- net ARD_D4: now also J9.8, U2.C2P021, U7.42; no longer J9.10, U2.C1P031, U7.38
- net ARD_D5: now also J9.6, U2.C3P024, U7.43; no longer J9.12, U2.3P000, U7.20GBIN3
- net DGND: now also J6.1, R41.1, SW1.1, SW6.1, SW7.1, SW8.1, T16.T, T23.T; no longer S1.1, S6.1, S7.1, S8.1
- net ICE_CRESETB: now also SW8.2; no longer S8.2
- net ICE_SDI: now also U7.14SPISO; no longer U7.17SPISI
- net ICE_SDO: now also U7.17SPISI; no longer U7.14SPISO
- net ICE_XTALEN: now also R41.2
- net N$11: now also SW6.2; no longer S6.2
- net N$12: now also SW7.S; no longer S7.S
- net N$13: now also SW1.S; no longer S1.S
- net N$14: now also SW6.S; no longer S6.S
- net N$16: now also SW8.S; no longer S8.S
- net N$9: now also SW7.2; no longer S7.2
- net NRF_AIN4: now also J9.4; no longer J9.14
- net NRF_AIN7: now also J9.2; no longer J9.16
- net NRF_LEDB: now also J3.1, R5.1; no longer J3.3, R7.1
- net NRF_LEDR: now also J3.3, R7.1; no longer J3.1, R5.1
- net NRF_RSTN: now also SW1.2; no longer S1.2
- net NRF_RXD: now also T19.T
- net NRF_SWDCLK: now also T18.T
- net NRF_SWDIO: now also T17.T
- net NRF_TXD: now also T20.T
- net NRF_USBCON5V: now also T24.T
- net NRF_USBDN: now also T21.T
- net NRF_USBDP: now also T22.T
- net STM_SWCLK: now also T27.T
- net STM_SWDIO: now also T14.T
- net UARTRX: now also J9.16; no longer J9.2
- net UARTTX: now also J9.14; no longer J9.4
Other:
- note removed: "need stronger pullup?"
- moved on the sheet: J4, T11, T12, T5, T6, T7, T8, T9
